File: hardware/avr-nrf.brd (EAGLE design)
At the start: 40 x 49 mm, 73 parts, among them IC2 MAX1555, J1 J0026, U1 ATMEGA32U2AU, U2 NRF24L01SMD, U3 USB-MINIB-5PIN, U4 KSZ8851SNL, Y1 16M, Y2 8M, Y3 25M

Commit message: hardware: fix eth cap values
Parts:
- C19: value 100u -> 10u
- C20, C21: value 10n -> .1u
Changed lines of the file:
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@@
 <?xml version="1.0" encoding="utf-8"?>
 <!DOCTYPE eagle SYSTEM "eagle.dtd">
-<eagle version="6.0">
+<eagle version="6.1">
 <drawing>
 <settings>
@@
 <element name="R16" library="rcl" package="R0603" value="330" x="23.7744" y="21.1328" rot="R90"/>
 <element name="R17" library="rcl" package="R0603" value="330" x="25.1968" y="21.1328" rot="R90"/>
-<element name="C19" library="rcl" package="C0805" value="100u" x="36.3728" y="21.1328" rot="R90"/>
+<element name="C19" library="rcl" package="C0805" value="10u" x="36.3728" y="21.1328" rot="R90"/>
 <element name="R18" library="rcl" package="R0603" value="50" x="31.496" y="21.1328" rot="R90"/>
-<element name="C20" library="rcl" package="C0805" value="10n" x="34.544" y="21.1328" rot="R90"/>
-<element name="C21" library="rcl" package="C0805" value="10n" x="26.8224" y="21.1328" rot="R90"/>
+<element name="C20" library="rcl" package="C0805" value=".1u" x="34.544" y="21.1328" rot="R90"/>
+<element name="C21" library="rcl" package="C0805" value=".1u" x="26.8224" y="21.1328" rot="R90"/>
 <element name="R19" library="rcl" package="R0603" value="50" x="32.9184" y="21.1328" rot="R90"/>
 <element name="R20" library="rcl" package="R0603" value="50" x="28.448" y="21.1328" rot="R90"/>

Commit message: hw: update antenna symbol on schematics
Parts:
- U$1: value INVERTED_F_ANTENNA -> INVERTED_F_ANTENNA+5; device antenna:DN007 -> antenna:DN007+5
Changed lines of the file:
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@@
 <attribute name="TP_SIGNAL_NAME" value="" x="11.3538" y="40.6908" size="1.778" layer="27" rot="R90" display="off"/>
 </element>
-<element name="U$1" library="antenna" package="DN007" value="INVERTED_F_ANTENNA" x="9.144" y="44.9072"/>
+<element name="U$1" library="antenna" package="DN007+5" value="INVERTED_F_ANTENNA+5" x="9.144" y="44.9072"/>
 <element name="U4" library="balto" package="MLF32-TH" value="KSZ8851SNL" x="30.48" y="28.0416"/>
 <element name="J1" library="micrel" package="PJ-J0" value="J0026" x="30.48" y="7.7216" rot="R180"/>
